File: Split 45.kicad_pcb (KiCad board)
At the start: 2 copper layers, 171 parts, among them SW1 SW_Push, SW2 SW_Push, U1 ATmega32U4-AU, U2 ATmega32U4-AU, Y1 16MHz, Y2 16MHz

Commit message: Place switch diodes
Parts:
- Y1, Y2: footprint Package_QFP:TQFP-44_10x10mm_P0.8mm -> Crystal:Crystal_SMD_3225-4Pin_3.2x2.5mm
- moved D60 472.0 mm to (412.0, 326.2), turned to 90 degrees
- moved D54 458.6 mm to (416.7, 307.2), turned to 90 degrees
- moved D59 437.8 mm to (376.2, 326.2), turned to 90 degrees
- moved D50 436.0 mm to (347.7, 307.2), turned to 90 degrees
- moved D53 432.1 mm to (390.5, 309.6)
- moved D52 425.6 mm to (385.8, 307.2), turned to 90 degrees
- moved D58 418.1 mm to (357.2, 326.2), turned to 90 degrees
- moved D57 398.9 mm to (338.1, 326.2), turned to 90 degrees
- moved D64 392.7 mm to (404.8, 345.3), turned to 90 degrees
- moved D51 389.2 mm to (366.7, 307.2), turned to 90 degrees
- moved MX_Enter2 386.8 mm to (417.5, 295.3)
- moved D56 380.3 mm to (319.1, 326.2), turned to 90 degrees
- moved D7 365.0 mm to (276.2, 269.1), turned to 90 degrees
- moved D63 362.6 mm to (376.2, 345.3), turned to 90 degrees
- moved D55 362.5 mm to (300.0, 326.2), turned to 90 degrees
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Connections:
- D7 pad 1: L_R0 -> R_R4
- MX_61 pad 1: L_C6 -> R_C3

Commit message: WIP routing
Parts:
- C1, C10, C11, C12, C13, C14, C2, C3, C4, C5, C6, C7, C8, C9, D1, D10, D11, D12, D13, D14, D15, D16, D17, D18, D19, D2, D20, D21, D22, D23, D24, D25, D26, D27, D28, D29, D3, D30, D31, D32, D33, D34, D35, D36, D37, D38, D39, D4, D40, D41, D42, D43, D44, D45, D46, D47, D48, D49, D5, D50, D51, D52, D53, D54, D55, D56, D57, D58, D59, D6, D60, D61, D62, D63, D64, D65, D7, D8, D9, F1, F2, R1, R2, R3, R4, R5, R6, R7, R8, SW1, USB1, USB2, Y1, Y2: moved to B.Cu
- U1, U2: footprint Package_QFP:TQFP-44_10x10mm_P0.8mm -> Package_DFN_QFN:QFN-44-1EP_7x7mm_P0.5mm_EP5.15x5.15mm; moved to B.Cu
- moved U2 365.8 mm to (325.3, 343.2), turned to 180 degrees
- moved Y2 365.2 mm to (327.0, 351.2)
- moved Y1 215.4 mm to (242.1, 484.2)
- moved USB2 202.2 mm to (354.0, 250.8), turned to 270 degrees
- moved U1 157.5 mm to (96.8, 396.1)
- moved C12 156.7 mm to (273.8, 498.5)
- moved USB1 138.9 mm to (53.2, 404.8)
- moved SW1 118.5 mm to (101.6, 447.7)
- moved MX_Plus1 114.3 mm to (381.8, 266.7)
- moved D7 114.3 mm to (390.5, 269.1)
- moved R8 107.5 mm to (338.9, 498.2)
- moved SW2 102.1 mm to (382.0, 339.0)
- moved C1 101.6 mm to (338.9, 495.3)
- moved C14 95.7 mm to (338.9, 492.4)
- moved R6 90.9 mm to (333.6, 340.9), turned to 90 degrees
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- renumbered MX_71 to MX_61, MX_81 to MX_71, MX_91 to MX_81, MX_Zero1 to MX_91, MX_Plus1 to MX_Minus1, MX_61 to MX_Plus1, MX_Minus1 to MX_Zero1
Connections:
- D26 pad 1: L_R3 -> L_R4
- D46 pad 1: R_R1 -> R_R2
- D54 pad 1: R_R2 -> R_R3
- D65 pad 1: R_R3 -> R_R4
- D7 pad 1: R_R4 -> R_R1
- MX_31 pad 1: Net-(MX_31-Pad1) -> L_C3
- MX_B1 pad 1: L_C6 -> L_C5
- MX_D1 pad 1: Net-(MX_D1-Pad1) -> L_C3
- MX_E1 pad 1: Net-(MX_E1-Pad1) -> L_C3
- MX_IsoSlash1 pad 1: L_C0 -> L_C1
- MX_LShift1 pad 1: L_C1 -> L_C0
- MX_LShift2 pad 1: L_C1 -> L_C0
- MX_X1 pad 1: Net-(MX_X1-Pad1) -> L_C3
- U1 pad 26: L_C6 -> Net-(U1-Pad26)
- U2 pad 12: Net-(U2-Pad12) -> R_R4
- U2 pad 28: R_R4 -> Net-(U2-Pad28)
Routing:
- net R_C3: track 0.00 -> 205.6 mm, vias 0 -> 1
- net R_R2: track 0.00 -> 151.8 mm, vias 0 -> 1
- net R_R3: track 0.00 -> 143.7 mm, vias 0 -> 1
- net R_R1: track 0.00 -> 119.5 mm, vias 0 -> 1
- net L_C2: track 0.00 -> 119.0 mm
- net R_C2: track 0.00 -> 116.3 mm, vias 0 -> 1
- net R_R4: track 0.00 -> 114.9 mm
- net L_C0: track 0.00 -> 114.7 mm
- net L_R4: track 0.00 -> 112.1 mm
- net R_C1: track 0.00 -> 111.9 mm, vias 0 -> 1
- net L_C4: track 0.00 -> 109.8 mm
- net L_R3: track 0.00 -> 109.5 mm
- net L_C1: track 0.00 -> 105.0 mm
- net L_R2: track 0.00 -> 102.4 mm
- net L_R1: track 0.00 -> 100.0 mm
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Other:
- net class Default: trace_width 0.25 -> 0.254
- net class Power added: clearance 0.2, trace_width 0.381, via_dia 0.8, via_drill 0.4

Commit message: Shitty work in progress
Parts:
- removed D7: D_Small, Diode_SMD:D_SOD-123
- removed the MX_HhkbTilde1 at (419.9, 266.7)
- added D66: D_Small, Diode_SMD:D_SOD-123, B.Cu at (428.4, 330.7)
- added D67: D_Schottky, random-keyboard-parts:D_SOD-123-Pretty, B.Cu at (377.3, 257.9)
- added ESD2: PRTR5V0U2X, random-keyboard-parts:SOT143B, B.Cu at (391.0, 262.9)
- added MX_Backslash1: MX-NoLED, MX_Only:MXOnly-1.5U-NoLED, F.Cu at (415.1, 285.8)
- added TRRS1: TRRS, random-keyboard-parts:PJ-3200B-4A, F.Cu at (3.43, 431.3)
- added TRRS2: TRRS, random-keyboard-parts:PJ-3200B-4A, F.Cu at (269.9, 254.0)
- MX_HhkbTilde1: renamed from MX_Backslash1; footprint MX_Only:MXOnly-1.5U-NoLED -> MX_Only:MXOnly-1U-NoLED
- U1, U2: footprint Package_DFN_QFN:QFN-44-1EP_7x7mm_P0.5mm_EP5.15x5.15mm -> Package_QFP:TQFP-44_10x10mm_P0.8mm
- moved C1 308.9 mm to (32.3, 458.1)
- moved C6 296.8 mm to (1.66, 472.0)
- moved C7 296.8 mm to (1.66, 474.9)
- moved C4 281.5 mm to (9.91, 474.7)
- moved R1 263.8 mm to (41.3, 457.6)
- moved R2 263.8 mm to (41.3, 454.6)
- moved R3 263.8 mm to (41.3, 451.7)
- moved R4 263.8 mm to (41.3, 448.7)
- moved C5 255.4 mm to (42.7, 444.9)
- moved C2 242.1 mm to (21.1, 464.9)
- moved F2 233.8 mm to (383.5, 257.9)
- moved C3 221.4 mm to (2.37, 458.1)
- moved F1 221.4 mm to (2.97, 461.2)
- moved Y1 189.2 mm to (54.3, 461.7)
- moved C12 175.2 mm to (323.0, 330.3), turned to 90 degrees
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Connections:
- net Net-(R5-Pad1) renamed R_Reset
- D46 pad 1: R_R2 -> R_R1
- D54 pad 1: R_R3 -> R_R2
- D65 pad 1: R_R4 -> R_R3
- F2 pad 1: +5V -> Net-(D67-Pad2)
- MX_Bksp1 pad 1: R_C6 -> R_C7
- MX_Bksp1 pad 2: Net-(D37-Pad2) -> Net-(D38-Pad2)
- MX_Enter1 pad 2: Net-(D54-Pad2) -> Net-(D65-Pad2)
- MX_Enter2 pad 2: Net-(D54-Pad2) -> Net-(D65-Pad2)
- MX_Fn1 pad 1: R_C7 -> R_C5
- MX_Fn1 pad 2: Net-(D65-Pad2) -> Net-(D66-Pad2)
- MX_HhkbBackslash1 pad 1: R_C6 -> R_C7
- MX_HhkbBackslash1 pad 2: Net-(D37-Pad2) -> Net-(D38-Pad2)
- MX_Plus1 pad 1: R_C3 -> R_C6
- MX_Plus1 pad 2: Net-(D7-Pad2) -> Net-(D37-Pad2)
- R6 pad 1: Net-(R6-Pad1) -> R_D+
- R6 pad 2: R_D+ -> Net-(ESD2-Pad2)
- R7 pad 1: Net-(R7-Pad1) -> R_D-
- R7 pad 2: R_D- -> Net-(ESD2-Pad3)
- U1 pad 10: L_R2 -> Net-(U1-Pad10)
- U1 pad 11: L_R3 -> Net-(U1-Pad11)
- U1 pad 18: L_C0 -> L_SCL
- U1 pad 19: L_C1 -> L_SDA
- U1 pad 20: L_C2 -> Net-(U1-Pad20)
- U1 pad 21: L_C3 -> Net-(U1-Pad21)
- U1 pad 22: L_C5 -> Net-(U1-Pad22)
- U1 pad 25: L_C4 -> Net-(U1-Pad25)
- U1 pad 28: L_R4 -> Net-(U1-Pad28)
- U1 pad 8: L_R0 -> Net-(U1-Pad8)
- U1 pad 9: L_R1 -> Net-(U1-Pad9)
- U2 pad 10: R_R2 -> Net-(U2-Pad10)
- U2 pad 11: R_R3 -> Net-(U2-Pad11)
- U2 pad 12: R_R4 -> Net-(U2-Pad12)
- U2 pad 18: R_C0 -> R_SCL
- U2 pad 19: R_C1 -> R_SDA
- U2 pad 20: R_C2 -> Net-(U2-Pad20)
- U2 pad 21: R_C3 -> Net-(U2-Pad21)
- U2 pad 22: R_C5 -> Net-(U2-Pad22)
- U2 pad 25: R_C4 -> R_R4
- U2 pad 26: R_C6 -> R_R3
- U2 pad 27: Net-(U2-Pad27) -> R_R2
- U2 pad 28: Net-(U2-Pad28) -> R_R1
- U2 pad 29: Net-(U2-Pad29) -> R_R0
- U2 pad 3: Net-(R7-Pad1) -> R_D-
- U2 pad 31: Net-(U2-Pad31) -> R_C5
- U2 pad 32: Net-(U2-Pad32) -> R_C6
- U2 pad 37: Net-(U2-Pad37) -> R_C0
- U2 pad 38: Net-(U2-Pad38) -> R_C1
- U2 pad 39: Net-(U2-Pad39) -> R_C2
- U2 pad 4: Net-(R6-Pad1) -> R_D+
- U2 pad 40: Net-(U2-Pad40) -> R_C3
- U2 pad 41: Net-(U2-Pad41) -> R_C4
- U2 pad 8: R_R0 -> Net-(U2-Pad8)
- U2 pad 9: R_R1 -> Net-(U2-Pad9)
- USB2 pad 3: R_D+ -> Net-(ESD2-Pad2)
- USB2 pad 4: R_D- -> Net-(ESD2-Pad3)
Routing:
- net GND: track 2.90 -> 384.8 mm, vias 0 -> 3
- net +5V: track 0.00 -> 324.3 mm, vias 0 -> 6
- net R_SDA: track 0.00 -> 125.8 mm, vias 0 -> 1
- net R_SCL: track 0.00 -> 121.3 mm, vias 0 -> 1
- net L_C2: track 119.0 -> 0.00 mm
- net R_D+: track 0.00 -> 115.5 mm
- net L_C0: track 114.7 -> 0.00 mm
- net R_D-: track 0.00 -> 113.5 mm
- net L_R4: track 112.1 -> 0.00 mm
- net L_C4: track 109.8 -> 0.00 mm
- net L_R3: track 109.5 -> 0.00 mm
- net L_C1: track 105.0 -> 0.00 mm
- net L_R2: track 102.4 -> 0.00 mm
- net L_R1: track 100.0 -> 0.00 mm
- net L_R0: track 95.2 -> 0.00 mm
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Other:
- board outline added: 173 x 106.4 mm
